Commit message: A bit of refactoring

File: urdf/macros/joint_components.xacro (robot description, xacro)
@@ -2,15 +2,15 @@
 <robot xmlns:xacro="http://www.ros.org/wiki/xacro">
     <!-- Hip joint properties: displacement and rotation relative to the base frame -->
-    <xacro:property name="hip_1_xyz" value="0.172664 0.092664 0.023" />
+    <xacro:property name="hip_1_xyz" value="0.172664 0.092664 0.0" />
     <xacro:property name="hip_1_rpy" value="0 0 ${pi/4}" />
-    <xacro:property name="hip_2_xyz" value="0.172664 -0.092664 0.023" />
+    <xacro:property name="hip_2_xyz" value="0.172664 -0.092664 0.0" />
     <xacro:property name="hip_2_rpy" value="0 0 ${-pi/4}" />
-    <xacro:property name="hip_3_xyz" value="0 0.12191 0.023" />
+    <xacro:property name="hip_3_xyz" value="0 0.12191 0.0" />
     <xacro:property name="hip_3_rpy" value="0 0 ${pi/2}" />
-    <xacro:property name="hip_4_xyz" value="0 -0.12191 0.023" />
+    <xacro:property name="hip_4_xyz" value="0 -0.12191 0.0" />
     <xacro:property name="hip_4_rpy" value="0 0 ${-pi/2}" />
-    <xacro:property name="hip_5_xyz" value="-0.172664 0.092664 0.023" />
+    <xacro:property name="hip_5_xyz" value="-0.172664 0.092664 0.0" />
     <xacro:property name="hip_5_rpy" value="0 0 ${3*pi/4}" />
-    <xacro:property name="hip_6_xyz" value="-0.172664 -0.092664 0.023" />
+    <xacro:property name="hip_6_xyz" value="-0.172664 -0.092664 0.0" />
     <xacro:property name="hip_6_rpy" value="0 0 ${-3*pi/4}" />
     <!-- Femur joint properties: displacement and rotation relative to the hip frame -->

File: urdf/macros/joints.xacro (robot description, xacro)
@@ -1,10 +1,12 @@
 <?xml version="1.0"?>
 <robot xmlns:xacro="http://www.ros.org/wiki/xacro">
-    <xacro:include filename="$(find neurowalker_description)/urdf/macros/joint_components.xacro" />
-    <joint name="dummy_joint" type="fixed">
-        <parent link="dummy_link" />
-        <child link="base_link" />
-        <origin xyz="0 0 0" rpy="0 0 0" />
-    </joint>
+    <xacro:include filename="joint_components.xacro" />
+    <xacro:if value="${kdl_compatible}">
+        <joint name="dummy_joint" type="fixed">
+            <parent link="dummy_link" />
+            <child link="base_link" />
+            <origin xyz="0 0 0" rpy="0 0 0" />
+        </joint>
+    </xacro:if>
     <xacro:hip_joint suffix="_1" use_joint_dynamics="${use_joint_dynamics}"/>
     <xacro:femur_joint suffix="_1" use_joint_dynamics="${use_joint_dynamics}" />

File: urdf/macros/link_components.xacro (robot description, xacro)
@@ -2,28 +2,16 @@
 <robot xmlns:xacro="http://www.ros.org/wiki/xacro">
     <!-- Full meshes file path -->
-    <xacro:property name="full_meshes"
-        value="package://neurowalker_description/meshes/full/stl" />
+    <xacro:property name="full_meshes" value="../../meshes/full/stl" />
     <!-- Simlpified meshes file path -->
-    <xacro:property name="simplified_meshes"
-        value="package://neurowalker_description/meshes/simplified/stl" />
-    <!-- Link colors. default_link_color applies to: base_link, hip_link, femur_link, tibia_link -->
-    <xacro:property name="default_link_color" value="0.79216 0.81961 0.93333 1" />
-    <xacro:property name="foot_tip_link_color"
-        value="0.694117647058824 0.0980392156862745 0.0980392156862745 1" />
+    <xacro:property name="simplified_meshes" value="../../meshes/simplified/stl" />
+    <!-- Link colors. robot_color applies to: base_link, hip_link, femur_link, tibia_link -->
+    <xacro:property name="robot_color" value="0.79216 0.81961 0.93333 1" />
+    <xacro:property name="foot_tip_color" value="0.694117647058824 0.0980392156862745 0.0980392156862745 1" />
     <xacro:macro name="base_link" params="simplify_meshes">
         <link name="base_link">
             <inertial>
-                <origin
-                    xyz="-3.8333E-17 -2.625E-17 0.02253"
-                    rpy="0 0 0" />
-                <mass
-                    value="1.0408" />
-                <inertia
-                    ixx="0.0011542"
-                    ixy="1.5544E-10"
-                    ixz="9.1238E-21"
-                    iyy="0.0039905"
-                    iyz="-2.7976E-20"
-                    izz="0.0049674" />
+                <origin xyz="-4.0647E-17 -2.3675E-17 -0.00046955" rpy="0 0 0" />
+                <mass value="1.0408" />
+                <inertia ixx="0.0011542" ixy="1.5544E-10" ixz="7.7333E-21" iyy="0.0039905" iyz="-3.097E-20" izz="0.0049674" />
             </inertial>
             <visual>
@@ -38,5 +26,5 @@
                 </geometry>
                 <material name="">
-                    <color rgba="${default_link_color}" />
+                    <color rgba="${robot_color}" />
                 </material>
             </visual>
@@ -57,16 +45,7 @@
         <link name="hip_link${suffix}">
             <inertial>
-                <origin
-                    xyz="0.0207539578220567 0.00016313993084466 -0.000157508593183945"
-                    rpy="0 0 0" />
-                <mass
-                    value="0.00976937887973851" />
-                <inertia
-                    ixx="4.36001352628253E-06"
-                    ixy="3.05074712305715E-11"
-                    ixz="1.09800410231598E-11"
-                    iyy="3.54065431889005E-06"
-                    iyz="-8.43037492910402E-22"
-                    izz="3.53980041929617E-06" />
+                <origin xyz="0.0207539578220567 0.00016313993084466 -0.000157508593183945" rpy="0 0 0" />
+                <mass value="0.00976937887973851" />
+                <inertia ixx="4.36001352628253E-06" ixy="3.05074712305715E-11" ixz="1.09800410231598E-11" iyy="3.54065431889005E-06" iyz="-8.43037492910402E-22" izz="3.53980041929617E-06" />
             </inertial>
             <visual>
@@ -81,5 +60,5 @@
                 </geometry>
                 <material name="">
-                    <color rgba="${default_link_color}" />
+                    <color rgba="${robot_color}" />
                 </material>
             </visual>
@@ -100,16 +79,7 @@
         <link name="femur_link${suffix}">
             <inertial>
-                <origin
-                    xyz="0.039 -0.000267065647974397 1.30227414534182E-05"
-                    rpy="0 0 0" />
-                <mass
-                    value="0.0681610759338743" />
-                <inertia
-                    ixx="1.22383085422276E-05"
-                    ixy="1.5544030901566E-10"
-                    ixz="2.33365338510496E-21"
-                    iyy="1.88790791713266E-05"
-                    iyz="1.60983936131494E-21"
-                    izz="1.12330386801315E-05" />
+                <origin xyz="0.039 -0.000267065647974397 1.30227414534182E-05" rpy="0 0 0" />
+                <mass value="0.0681610759338743" />
+                <inertia ixx="1.22383085422276E-05" ixy="1.5544030901566E-10" ixz="2.33365338510496E-21" iyy="1.88790791713266E-05" iyz="1.60983936131494E-21" izz="1.12330386801315E-05" />
             </inertial>
             <visual>
@@ -124,5 +94,5 @@
                 </geometry>
                 <material name="">
-                    <color rgba="${default_link_color}" />
+                    <color rgba="${robot_color}" />
                 </material>
             </visual>
@@ -143,16 +113,7 @@
         <link name="tibia_link${suffix}">
             <inertial>
-                <origin
-                    xyz="0.0863740398095008 -0.0136567529957215 2.8854666747154E-08"
-                    rpy="0 0 0" />
-                <mass
-                    value="0.0518953116111732" />
-                <inertia
-                    ixx="2.14028837547244E-05"
-                    ixy="1.20884063145876E-05"
-                    ixz="3.60427983546376E-11"
-                    iyy="5.18668393911014E-05"
-                    iyz="-1.36891234811654E-11"
-                    izz="4.38855876942104E-05" />
+                <origin xyz="0.0863740398095008 -0.0136567529957215 2.8854666747154E-08" rpy="0 0 0" />
+                <mass value="0.0518953116111732" />
+                <inertia ixx="2.14028837547244E-05" ixy="1.20884063145876E-05" ixz="3.60427983546376E-11" iyy="5.18668393911014E-05" iyz="-1.36891234811654E-11" izz="4.38855876942104E-05" />
             </inertial>
             <visual>
@@ -167,5 +128,5 @@
                 </geometry>
                 <material name="">
-                    <color rgba="${default_link_color}" />
+                    <color rgba="${robot_color}" />
                 </material>
             </visual>
@@ -186,16 +147,7 @@
         <link name="foot_tip_link${suffix}">
             <inertial>
-                <origin
-                    xyz="0.00119417475728155 9.48943996844099E-20 -1.38897240469442E-19"
-                    rpy="0 0 0" />
-                <mass
-                    value="0.00345156312874398" />
-                <inertia
-                    ixx="1.55434275887049E-07"
-                    ixy="-1.7646776450454E-24"
-                    ixz="-3.90368160252396E-24"
-                    iyy="1.2879747429975E-07"
-                    iyz="-6.17628190706261E-24"
-                    izz="1.2879747429975E-07" />
+                <origin xyz="0.00119417475728155 9.48943996844099E-20 -1.38897240469442E-19" rpy="0 0 0" />
+                <mass value="0.00345156312874398" />
+                <inertia ixx="1.55434275887049E-07" ixy="-1.7646776450454E-24" ixz="-3.90368160252396E-24" iyy="1.2879747429975E-07" iyz="-6.17628190706261E-24" izz="1.2879747429975E-07" />
             </inertial>
             <visual>
@@ -210,5 +162,5 @@
                 </geometry>
                 <material name="">
-                    <color rgba="${foot_tip_link_color}" />
+                    <color rgba="${foot_tip_color}" />
                 </material>
             </visual>

File: urdf/macros/links.xacro (robot description, xacro)
@@ -1,6 +1,8 @@
 <?xml version="1.0"?>
 <robot xmlns:xacro="http://www.ros.org/wiki/xacro">
-    <xacro:include filename="$(find neurowalker_description)/urdf/macros/link_components.xacro" />
-    <link name="dummy_link" />
+    <xacro:include filename="link_components.xacro" />
+    <xacro:if value="${kdl_compatible}">
+        <link name="dummy_link" />
+    </xacro:if>
     <xacro:base_link simplify_meshes="${simplify_meshes}" />
     <xacro:hip_link suffix="_1" simplify_meshes="${simplify_meshes}" />

File: urdf/neurowalker.xacro (robot description, xacro)
@@ -1,13 +1,16 @@
 <?xml version="1.0"?>
 <robot name="neurowalker" xmlns:xacro="http://www.ros.org/wiki/xacro">
+    <!-- Define whether to generate KDL compatible URDF (Extra dummy link without inertia properties) -->
+    <xacro:arg name="kdl_compatible" default="false" />
+    <xacro:property name="kdl_compatible" value="$(arg kdl_compatible)" />
     <!-- Include robot links -->
     <!-- Define whether to use simplified meshes -->
     <xacro:arg name="simplify_meshes" default="true" />
     <xacro:property name="simplify_meshes" value="$(arg simplify_meshes)" />
-    <xacro:include filename="$(find neurowalker_description)/urdf/macros/links.xacro" />
+    <xacro:include filename="macros/links.xacro" />
     <!-- Include robot joints -->
     <!-- Define whether to use joint dynamics. In this package it doesnt matter -->
     <xacro:arg name="use_joint_dynamics" default="false" />
     <xacro:property name="use_joint_dynamics" value="$(arg use_joint_dynamics)" />
-    <xacro:include filename="$(find neurowalker_description)/urdf/macros/joints.xacro" />
+    <xacro:include filename="macros/joints.xacro" />
 </robot>

Commit message: Final refactoring

File: urdf/macros/joint_components.xacro (robot description, xacro)
@@ -23,12 +23,12 @@
     <xacro:property name="foot_tip_xyz" value="${0.0515+0.106*cos(-pi/9)} ${0.106*sin(-pi/9)} 0" />
     <xacro:property name="foot_tip_rpy" value="0 0 ${-pi/9}" />
-    <!-- Servo limitations -->
-    <xacro:property name="servo_lower" value="${-2*pi/3}" />
-    <xacro:property name="servo_upper" value="${2*pi/3}" />
-    <xacro:property name="servo_velocity" value="5.8178" />
-    <xacro:property name="servo_effort" value="1.9613" />
-    <xacro:macro name="servo_limit">
-        <limit lower="${servo_lower}" upper="${servo_upper}" velocity="${servo_velocity}"
-            effort="${servo_effort}" />
+    <!-- Servo physical limitations -->
+    <xacro:property name="servo_physical_lower" value="${-2*pi/3}" />
+    <xacro:property name="servo_physical_upper" value="${2*pi/3}" />
+    <xacro:property name="servo_physical_velocity" value="5.8178" />
+    <xacro:property name="servo_physical_effort" value="1.9613" />
+    <xacro:macro name="servo_physical_limit">
+        <limit lower="${servo_physical_lower}" upper="${servo_physical_upper}" velocity="${servo_physical_velocity}"
+            effort="${servo_physical_effort}" />
     </xacro:macro>
     <!-- Servo dynamics. Some random values right now -->
@@ -62,5 +62,5 @@
             </xacro:if>
             <axis xyz="0 0 1" />
-            <xacro:servo_limit />
+            <xacro:servo_physical_limit />
             <xacro:if value="${use_joint_dynamics}">
                 <xacro:joint_dynamics />
@@ -75,5 +75,5 @@
             <origin xyz="${femur_xyz}" rpy="${femur_rpy}" />
             <axis xyz="0 0 1" />
-            <xacro:servo_limit />
+            <xacro:servo_physical_limit />
             <xacro:if value="${use_joint_dynamics}">
                 <xacro:joint_dynamics />
@@ -88,5 +88,5 @@
             <origin xyz="${tibia_xyz}" rpy="${tibia_rpy}" />
             <axis xyz="0 0 1" />
-            <xacro:servo_limit />
+            <xacro:servo_physical_limit />
             <xacro:if value="${use_joint_dynamics}">
                 <xacro:joint_dynamics />

File: urdf/macros/link_components.xacro (robot description, xacro)
@@ -2,7 +2,7 @@
 <robot xmlns:xacro="http://www.ros.org/wiki/xacro">
     <!-- Full meshes file path -->
-    <xacro:property name="full_meshes" value="../../meshes/full/stl" />
+    <xacro:property name="full_meshes" value="../meshes/full/stl" />
     <!-- Simlpified meshes file path -->
-    <xacro:property name="simplified_meshes" value="../../meshes/simplified/stl" />
+    <xacro:property name="simplified_meshes" value="../meshes/simplified/stl" />
     <!-- Link colors. robot_color applies to: base_link, hip_link, femur_link, tibia_link -->
     <xacro:property name="robot_color" value="0.79216 0.81961 0.93333 1" />

File: urdf/neurowalker.urdf (robot description, URDF)
Before this commit: robot neurowalker, 25 links, 24 joints
Links:
- link base_link: geometry collision mesh filename=../meshes/simplified/stl/base_link.STL; visual mesh filename=../meshes/simplified/stl/base_link.STL
- link femur_link_1: geometry collision mesh filename=../meshes/simplified/stl/femur_link.STL; visual mesh filename=../meshes/simplified/stl/femur_link.STL
- link femur_link_2: geometry collision mesh filename=../meshes/simplified/stl/femur_link.STL; visual mesh filename=../meshes/simplified/stl/femur_link.STL
- link femur_link_3: geometry collision mesh filename=../meshes/simplified/stl/femur_link.STL; visual mesh filename=../meshes/simplified/stl/femur_link.STL
- link femur_link_4: geometry collision mesh filename=../meshes/simplified/stl/femur_link.STL; visual mesh filename=../meshes/simplified/stl/femur_link.STL
- link femur_link_5: geometry collision mesh filename=../meshes/simplified/stl/femur_link.STL; visual mesh filename=../meshes/simplified/stl/femur_link.STL
- link femur_link_6: geometry collision mesh filename=../meshes/simplified/stl/femur_link.STL; visual mesh filename=../meshes/simplified/stl/femur_link.STL
- link foot_tip_link_1: geometry collision mesh filename=../meshes/simplified/stl/foot_tip_link.STL; visual mesh filename=../meshes/simplified/stl/foot_tip_link.STL
- link foot_tip_link_2: geometry collision mesh filename=../meshes/simplified/stl/foot_tip_link.STL; visual mesh filename=../meshes/simplified/stl/foot_tip_link.STL
- link foot_tip_link_3: geometry collision mesh filename=../meshes/simplified/stl/foot_tip_link.STL; visual mesh filename=../meshes/simplified/stl/foot_tip_link.STL
- link foot_tip_link_4: geometry collision mesh filename=../meshes/simplified/stl/foot_tip_link.STL; visual mesh filename=../meshes/simplified/stl/foot_tip_link.STL
- link foot_tip_link_5: geometry collision mesh filename=../meshes/simplified/stl/foot_tip_link.STL; visual mesh filename=../meshes/simplified/stl/foot_tip_link.STL
- link foot_tip_link_6: geometry collision mesh filename=../meshes/simplified/stl/foot_tip_link.STL; visual mesh filename=../meshes/simplified/stl/foot_tip_link.STL
- link hip_link_1: geometry collision mesh filename=../meshes/simplified/stl/hip_link.STL; visual mesh filename=../meshes/simplified/stl/hip_link.STL
- link hip_link_2: geometry collision mesh filename=../meshes/simplified/stl/hip_link.STL; visual mesh filename=../meshes/simplified/stl/hip_link.STL
- link hip_link_3: geometry collision mesh filename=../meshes/simplified/stl/hip_link.STL; visual mesh filename=../meshes/simplified/stl/hip_link.STL
- link hip_link_4: geometry collision mesh filename=../meshes/simplified/stl/hip_link.STL; visual mesh filename=../meshes/simplified/stl/hip_link.STL
- link hip_link_5: geometry collision mesh filename=../meshes/simplified/stl/hip_link.STL; visual mesh filename=../meshes/simplified/stl/hip_link.STL
- link hip_link_6: geometry collision mesh filename=../meshes/simplified/stl/hip_link.STL; visual mesh filename=../meshes/simplified/stl/hip_link.STL
- link tibia_link_1: geometry collision mesh filename=../meshes/simplified/stl/tibia_link.STL; visual mesh filename=../meshes/simplified/stl/tibia_link.STL
- link tibia_link_2: geometry collision mesh filename=../meshes/simplified/stl/tibia_link.STL; visual mesh filename=../meshes/simplified/stl/tibia_link.STL
- link tibia_link_3: geometry collision mesh filename=../meshes/simplified/stl/tibia_link.STL; visual mesh filename=../meshes/simplified/stl/tibia_link.STL
- link tibia_link_4: geometry collision mesh filename=../meshes/simplified/stl/tibia_link.STL; visual mesh filename=../meshes/simplified/stl/tibia_link.STL
- link tibia_link_5: geometry collision mesh filename=../meshes/simplified/stl/tibia_link.STL; visual mesh filename=../meshes/simplified/stl/tibia_link.STL
- link tibia_link_6: geometry collision mesh filename=../meshes/simplified/stl/tibia_link.STL; visual mesh filename=../meshes/simplified/stl/tibia_link.STL

File: urdf/neurowalker.xacro (robot description, xacro)
@@ -1,14 +1,14 @@
 <?xml version="1.0"?>
 <robot name="neurowalker" xmlns:xacro="http://www.ros.org/wiki/xacro">
-    <!-- Define whether to generate KDL compatible URDF (Extra dummy link without inertia properties) -->
+    <!-- Choose whether to generate KDL compatible URDF (Extra dummy link without inertia properties) -->
     <xacro:arg name="kdl_compatible" default="false" />
     <xacro:property name="kdl_compatible" value="$(arg kdl_compatible)" />
     <!-- Include robot links -->
-    <!-- Define whether to use simplified meshes -->
-    <xacro:arg name="simplify_meshes" default="true" />
+    <!-- Choose whether to use simplified meshes -->
+    <xacro:arg name="simplify_meshes" default="false" />
     <xacro:property name="simplify_meshes" value="$(arg simplify_meshes)" />
     <xacro:include filename="macros/links.xacro" />
     <!-- Include robot joints -->
-    <!-- Define whether to use joint dynamics. In this package it doesnt matter -->
+    <!-- Choose whether to add dynamics tag. In this package it doesnt matter -->
     <xacro:arg name="use_joint_dynamics" default="false" />
     <xacro:property name="use_joint_dynamics" value="$(arg use_joint_dynamics)" />
