Commit message: minor changes

File: urdf/macros/joint_components.xacro (robot description, xacro)
@@ -23,12 +23,16 @@
     <xacro:property name="foot_tip_xyz" value="${0.0515+0.106*cos(-pi/9)} ${0.106*sin(-pi/9)} 0" />
     <xacro:property name="foot_tip_rpy" value="0 0 ${-pi/9}" />
-    <!-- Servo physical limitations -->
-    <xacro:property name="servo_physical_lower" value="${-2*pi/3}" />
-    <xacro:property name="servo_physical_upper" value="${2*pi/3}" />
-    <xacro:property name="servo_physical_velocity" value="5.8178" />
-    <xacro:property name="servo_physical_effort" value="1.9613" />
-    <xacro:macro name="servo_physical_limit">
-        <limit lower="${servo_physical_lower}" upper="${servo_physical_upper}" velocity="${servo_physical_velocity}"
-            effort="${servo_physical_effort}" />
+    <!-- Servo limits -->
+    <xacro:property name="velocity_limit" value="5.8178" />
+    <xacro:property name="effort_limit" value="1.9613" />
+    <xacro:property name="servo_lower_limit" value="${-2*pi/3}" />
+    <xacro:property name="servo_upper_limit" value="${2*pi/3}" />
+    <xacro:macro name="hip_limit">
+        <limit lower="${-pi/2}" upper="${pi/2}" velocity="${velocity_limit}"
+            effort="${effort_limit}" />
+    </xacro:macro>
+    <xacro:macro name="servo_limit">
+        <limit lower="${servo_lower_limit}" upper="${servo_upper_limit}" velocity="${velocity_limit}"
+            effort="${effort_limit}" />
     </xacro:macro>
     <!-- Servo dynamics. Some random values right now -->
@@ -62,5 +66,5 @@
             </xacro:if>
             <axis xyz="0 0 1" />
-            <xacro:servo_physical_limit />
+            <xacro:hip_limit />
             <xacro:if value="${use_joint_dynamics}">
                 <xacro:joint_dynamics />
@@ -75,5 +79,5 @@
             <origin xyz="${femur_xyz}" rpy="${femur_rpy}" />
             <axis xyz="0 0 1" />
-            <xacro:servo_physical_limit />
+            <xacro:servo_limit />
             <xacro:if value="${use_joint_dynamics}">
                 <xacro:joint_dynamics />
@@ -88,5 +92,5 @@
             <origin xyz="${tibia_xyz}" rpy="${tibia_rpy}" />
             <axis xyz="0 0 1" />
-            <xacro:servo_physical_limit />
+            <xacro:servo_limit />
             <xacro:if value="${use_joint_dynamics}">
                 <xacro:joint_dynamics />

File: urdf/neurowalker.urdf (robot description, URDF)
Before this commit: robot neurowalker, 25 links, 24 joints
Joints:
- joint hip_joint_1: limit lower=-2.0943951023931953 upper=2.0943951023931953 effort=1.9613 velocity=5.8178 -> lower=-1.5707963267948966 upper=1.5707963267948966 effort=1.9613 velocity=5.8178
- joint hip_joint_2: limit lower=-2.0943951023931953 upper=2.0943951023931953 effort=1.9613 velocity=5.8178 -> lower=-1.5707963267948966 upper=1.5707963267948966 effort=1.9613 velocity=5.8178
- joint hip_joint_3: limit lower=-2.0943951023931953 upper=2.0943951023931953 effort=1.9613 velocity=5.8178 -> lower=-1.5707963267948966 upper=1.5707963267948966 effort=1.9613 velocity=5.8178
- joint hip_joint_4: limit lower=-2.0943951023931953 upper=2.0943951023931953 effort=1.9613 velocity=5.8178 -> lower=-1.5707963267948966 upper=1.5707963267948966 effort=1.9613 velocity=5.8178
- joint hip_joint_5: limit lower=-2.0943951023931953 upper=2.0943951023931953 effort=1.9613 velocity=5.8178 -> lower=-1.5707963267948966 upper=1.5707963267948966 effort=1.9613 velocity=5.8178
- joint hip_joint_6: limit lower=-2.0943951023931953 upper=2.0943951023931953 effort=1.9613 velocity=5.8178 -> lower=-1.5707963267948966 upper=1.5707963267948966 effort=1.9613 velocity=5.8178

File: urdf/neurowalker.xacro (robot description, xacro)
@@ -6,5 +6,5 @@
     <!-- Include robot links -->
     <!-- Choose whether to use simplified meshes -->
-    <xacro:arg name="simplify_meshes" default="false" />
+    <xacro:arg name="simplify_meshes" default="true" />
     <xacro:property name="simplify_meshes" value="$(arg simplify_meshes)" />
     <xacro:include filename="macros/links.xacro" />
